Commit message: created web_server pkg

File: src/robot_description/model/robot_1.urdf (robot description, URDF)
Before this commit: robot rover, 9 links, 8 joints
Links:
- added link ultrasonic_back_emission; visual sphere radius=0.005
- added link ultrasonic_front_emission; visual sphere radius=0.005
Joints:
- added joint ultrasonic_back_emission_point: type fixed, parent base_link, child ultrasonic_back_emission, origin xyz=0 -0.125 0.0 rpy=0 0 3.141592654, axis 1 1 1
- added joint ultrasonic_front_emission_point: type fixed, parent base_link, child ultrasonic_front_emission, origin xyz=0 0.125 0.0 rpy=0 0 0, axis 1 1 1

Commit message: Added laser scan sim to sensor drivers

File: src/robot_description/model/robot_1.urdf (robot description, URDF)
Before this commit: robot rover, 11 links, 10 joints
Links:
- removed link ultrasonic_back_emission
- removed link ultrasonic_front_emission
- added link laser_scan_center_point; visual sphere radius=0.01
- added link ultrasonic_back_emission_point; visual sphere radius=0.01
- added link ultrasonic_front_emission_point; visual sphere radius=0.01
- added link ultrasonic_left_emission_point; visual sphere radius=0.01
- added link ultrasonic_right_emission_point; visual sphere radius=0.01
Joints:
- removed joint ultrasonic_back_emission_point
- removed joint ultrasonic_front_emission_point
- added joint laser_scan_center_joint: type fixed, parent base_link, child laser_scan_center_point, origin xyz=0 0 -0.011 rpy=0 0 0, axis 1 1 1
- added joint ultrasonic_back_emission_joint: type fixed, parent base_link, child ultrasonic_back_emission_point, origin xyz=0 -0.11 -0.011 rpy=0 0 -1.57079632679, axis 1 1 1
- added joint ultrasonic_front_emission_joint: type fixed, parent base_link, child ultrasonic_front_emission_point, origin xyz=0 0.11 -0.011 rpy=0 0 1.57079632679, axis 1 1 1
- added joint ultrasonic_left_emission_joint: type fixed, parent base_link, child ultrasonic_left_emission_point, origin xyz=-0.085 0.086 -0.011 rpy=0 0 3.141592654, axis 1 1 1
- added joint ultrasonic_right_emission_joint: type fixed, parent base_link, child ultrasonic_right_emission_point, origin xyz=0.085 0.086 -0.011 rpy=0 0 0, axis 1 1 1

Commit message: Update robot_1.urdf

File: src/robot_description/model/robot_1.urdf (robot description, URDF)
Before this commit: robot rover, 14 links, 13 joints
Links:
- removed link caster
- added link left_caster; visual sphere radius=0.017
- added link right_caster; visual sphere radius=0.017
- link base_link: geometry visual box size=0.18 0.18 0.051
Joints:
- removed joint caster_joint
- added joint left_caster_joint: type fixed, parent base_link, child left_caster, origin xyz=-0.05 -0.07 -0.0235 rpy=0 0 0, axis 1 1 1
- added joint right_caster_joint: type fixed, parent base_link, child right_caster, origin xyz=0.05 -0.07 -0.0235 rpy=0 0 0, axis 1 1 1
- joint ultrasonic_back_emission_joint: origin xyz=0 -0.11 -0.011 rpy=0 0 -1.57079632679 -> xyz=0 -0.075 -0.011 rpy=0 0 -1.57079632679
- joint ultrasonic_back_joint: origin xyz=0 -0.11 -0.011 rpy=0 0 3.141592654 -> xyz=0 -0.075 -0.011 rpy=0 0 3.141592654
- joint ultrasonic_front_emission_joint: origin xyz=0 0.11 -0.011 rpy=0 0 1.57079632679 -> xyz=0 0.075 -0.011 rpy=0 0 1.57079632679
- joint ultrasonic_front_joint: origin xyz=0 0.11 -0.011 rpy=0 0 0 -> xyz=0 0.075 -0.011 rpy=0 0 0
- joint ultrasonic_left_emission_joint: origin xyz=-0.085 0.086 -0.011 rpy=0 0 3.141592654 -> xyz=-0.075 0.0395 -0.011 rpy=0 0 3.141592654
- joint ultrasonic_left_joint: origin xyz=-0.085 0.086 -0.011 rpy=0 0 1.57079632679 -> xyz=-0.075 0.0395 -0.011 rpy=0 0 1.57079632679
- joint ultrasonic_right_emission_joint: origin xyz=0.085 0.086 -0.011 rpy=0 0 0 -> xyz=0.075 0.0395 -0.011 rpy=0 0 0
- joint ultrasonic_right_joint: origin xyz=0.085 0.086 -0.011 rpy=0 0 -1.57079632679 -> xyz=0.075 0.0395 -0.011 rpy=0 0 -1.57079632679
- joint wheel_left_joint: origin xyz=-0.0914 -0.0775 -.0105 rpy=1.57079632679 0 1.57079632679 -> xyz=-0.0857 0.0485 -.0105 rpy=1.57079632679 0 1.57079632679
- joint wheel_right_joint: origin xyz=0.0914 -0.0775 -.0105 rpy=1.57079632679 0 1.57079632679 -> xyz=0.0857 0.0485 -.0105 rpy=1.57079632679 0 1.57079632679

Commit message: added pull to start

File: src/robot_description/model/robot_1.urdf (robot description, URDF)
Before this commit: robot rover, 15 links, 14 joints
Links:
- added link robot_center; visual box size=0.18 0.18 0.051
- link base_link: geometry 
Joints:
- added joint robot_center_joint: type fixed, parent base_link, child robot_center, origin xyz=0 -0.0485 0 rpy=0 0 0, axis 1 1 1
- joint head_indication_joint: parent base_link -> robot_center
- joint laser_scan_center_joint: parent base_link -> robot_center
- joint left_caster_joint: parent base_link -> robot_center
- joint right_caster_joint: parent base_link -> robot_center
- joint ultrasonic_back_emission_joint: parent base_link -> robot_center
- joint ultrasonic_back_joint: parent base_link -> robot_center
- joint ultrasonic_front_emission_joint: parent base_link -> robot_center
- joint ultrasonic_front_joint: parent base_link -> robot_center
- joint ultrasonic_left_emission_joint: origin xyz=-0.075 0.0395 -0.011 rpy=0 0 3.141592654 -> xyz=-0.075 -0.0395 -0.011 rpy=0 0 3.141592654; parent base_link -> robot_center
- joint ultrasonic_left_joint: origin xyz=-0.075 0.0395 -0.011 rpy=0 0 1.57079632679 -> xyz=-0.075 -0.0395 -0.011 rpy=0 0 1.57079632679; parent base_link -> robot_center
- joint ultrasonic_right_emission_joint: origin xyz=0.075 0.0395 -0.011 rpy=0 0 0 -> xyz=0.075 -0.0395 -0.011 rpy=0 0 0; parent base_link -> robot_center
- joint ultrasonic_right_joint: origin xyz=0.075 0.0395 -0.011 rpy=0 0 -1.57079632679 -> xyz=0.075 -0.0395 -0.011 rpy=0 0 -1.57079632679; parent base_link -> robot_center
- joint wheel_left_joint: parent base_link -> robot_center
- joint wheel_right_joint: parent base_link -> robot_center
